Commit message: new robot model

File: urdf/turtle_macros.xacro (robot description, xacro)
@@ -22,4 +22,9 @@
                 <origin xyz="0 0 0" rpy="0 0 0"/>
             </collision>
+            <inertial>
+                <mass value="0.1" />
+                <origin xyz="0 0 0" />
+                <inertia ixx="0.0001" ixy="0.0" ixz="0.0" iyy="0.0001" iyz="0.0" izz="0.0001" />
+            </inertial>
         </link>
     </xacro:macro>
@@ -33,4 +38,9 @@
                 <material name="${color}"/>
             </visual>
+            <inertial>
+                <mass value="0.1" />
+                <origin xyz="0 0 0" />
+                <inertia ixx="0.0001" ixy="0.0" ixz="0.0" iyy="0.0001" iyz="0.0" izz="0.0001" />
+            </inertial>
         </link>
         <joint name="${prefix}_wheel_joint" type="continuous">
@@ -54,4 +64,9 @@
                 <material name="${name}_material"><color rgba="${color_rgba}"/></material>
             </visual>
+            <inertial>
+                <mass value="0.1" />
+                <origin xyz="0 0 0" />
+                <inertia ixx="0.0001" ixy="0.0" ixz="0.0" iyy="0.0001" iyz="0.0" izz="0.0001" />
+            </inertial>
         </link>
         <joint name="${name}_joint" type="fixed">
