Commit message: moving the robot up

File: urdf/robot.urdf (robot description, URDF)
Before this commit: robot diff_drive_robot, 7 links, 6 joints
Joints:
- joint chassis_joint: origin xyz=-0.1 0 0 -> xyz=-0.1 0 0.05
- joint left_wheel_joint: origin xyz=0 0.175 0 rpy=-${pi/2} 0 0 -> xyz=0 0.175 0.05 rpy=-${pi/2} 0 0
- joint right_wheel_joint: origin xyz=0 -0.175 0 rpy=${pi/2} 0 0 -> xyz=0 -0.175 0.05 rpy=${pi/2} 0 0

Commit message: adding point cloud sensor

File: urdf/robot.urdf (robot description, URDF)
Before this commit: robot diff_drive_robot, 7 links, 6 joints
Links:
- added link point_cloud_frame; collision box size=0.05 0.05 0.05; visual box size=0.05 0.05 0.05
Joints:
- added joint point_cloud_joint: type fixed, parent chassis, child point_cloud_frame, origin xyz=0.15 0.0 0.05 rpy=0 0 0
